Commit message: Baselines policy training allergo hand face down dex manipulation

File: assets/urdf/table_small.urdf (robot description, URDF)
Before this commit: robot object, 1 links, 0 joints
Links:
- removed link object
- added link box, mass 500; collision box size=0.12 0.12 0.5; visual box size=0.12 0.12 0.5
