Commit message: allergo hand and shadow hand baseline env

File: assets/urdf/allegro_hand_v4/allegro_hand_description/allegro_hand_right_move_base.urdf (robot description, URDF)
Before this commit: robot allegro_hand_right, 25 links, 24 joints
Joints:
- joint base_x_to_base_y: limit lower=-0.03 upper=0.03 effort=50 velocity=0.5 -> lower=-0.01 upper=0.01 effort=0.5 velocity=0.5
- joint base_y_to_base_z: limit lower=-0.03 upper=0.03 effort=50 velocity=0.5 -> lower=-0.01 upper=0.01 effort=0.5 velocity=0.5
- joint root_to_base_x: limit lower=-0.03 upper=0.03 effort=50 velocity=0.5 -> lower=-0.01 upper=0.01 effort=0.5 velocity=0.5

File: assets/urdf/objects/cube_multicolor.urdf (robot description, URDF)
Before this commit: robot object, 1 links, 0 joints
Links:
- link object: geometry collision box size=0.055 0.055 0.055; visual mesh filename=meshes/cube_multicolor.obj scale=.055 .055 .055

File: assets/urdf/objects/cube_multicolor_allegro.urdf (robot description, URDF)
Before this commit: robot object, 1 links, 0 joints
Links:
- link object: geometry collision box size=0.055 0.055 0.055; visual mesh filename=meshes/cube_multicolor.obj scale=.055 .055 .055
