Commit message: update with initial pose penalty

File: assets/urdf/objects/cylinder.urdf (robot description, URDF)
Before this commit: robot object, 1 links, 0 joints
Links:
- link object: geometry collision mesh filename=meshes/set_obj11_cylinder_0decompose.obj scale=.035 .035 .035; visual mesh filename=meshes/set_obj11_cylinder.obj scale=.035 .035 .035
